File: Loads_Control.kicad_sch (KiCad schematic)
At the start: 22 parts, among them J1 Conn_01x04_Pin, Q1 STN3NF06, Q2 BC817, Q3 BC817, Q4 STN3NF06, Q5 BC817, Q6 STN3NF06

Commit message: Lesson 4 - Power Supply
Parts:
- added D3: D, Diode_SMD:D_SOD-123F, symbol Device:D
- added J2, J3: Conn_01x01_Socket, MountingHole:MountingHole_3mm_Pad_Via, symbol Connector:Conn_01x01_Socket
- added K1: G2RL-1A-H, Relay_THT:Relay_SPST_Omron_G2RL-1A, symbol Relay:G2RL-1A-H
- added Q7: BC817, Package_TO_SOT_SMD:SOT-23, symbol Transistor_BJT:BC817
- added R18: 1k, Resistor_SMD:R_1206_3216Metric, symbol Device:R
- added R19: 10k, Resistor_SMD:R_1206_3216Metric, symbol Device:R
Connections:
- net +12V: now also D3.1 (K), K1.A1
- net GND: now also Q7.2 (E), R19.1
- new net: J3.1 (Pin_1), K1.13
- new net: Q7.1 (B), R18.2, R19.2
- new net: J2.1 (Pin_1), K1.14
- new net: D3.2 (A), K1.A2, Q7.3 (C)
- new net RELAY: R18.1
Other:
- moved on the sheet: J1
