File: Bluetooth_Module.kicad_pcb (KiCad board)
At the start: 2 copper layers, 60.5 x 61.4 mm, 45 parts, among them J1 Conn_01x04_Pin, J2 Conn_01x01_Socket, J3 Conn_01x01_Socket, J4 Jack-DC, K1 G2RL-1A-H, Q1 STN3NF06, Q2 BC817, Q3 BC817, Q4 STN3NF06, Q5 BC817, Q6 STN3NF06, Q7 BC817, U1 ESP32-C3-DevKitM-1

Commit message: Final version, gerbers generated
Parts:
- removed H3: MountingHole, MountingHole:MountingHole_3.5mm
- added C6: 1u/6V3, Capacitor_SMD:C_1206_3216Metric, F.Cu at (95.5, 64.6)
- R12, R17, R7: value 1k -> 100k
- moved D1 21.1 mm to (124.2, 85.1), turned to 180 degrees
- moved Q7 18.1 mm to (144.2, 70.7), turned to -90 degrees
- moved D2 17.8 mm to (124.2, 87.9), turned to 180 degrees
- moved R2 7.10 mm to (110.4, 90.3), turned to 180 degrees
- moved R1 6.44 mm to (110.2, 85.1), turned to 180 degrees
- moved R17 5.64 mm to (145.2, 55.1), turned to 90 degrees
- moved R16 4.64 mm to (144.2, 61.8)
- moved R15 4.32 mm to (144.2, 64.5)
- moved R19 2.73 mm to (117.7, 93.8), turned to 90 degrees
- moved R12 2.34 mm to (128.1, 61.7)
- moved C5 1.84 mm to (95.5, 61.6)
- moved Q6 1.80 mm to (137.7, 60.2)
- moved R18 1.60 mm to (118.7, 89.7)
- moved R13 0.35 mm to (137.7, 73.0)
Connections:
- J1 pad 1: unconnected-(J1-Pin_1-Pad1) -> LED_B_OUT
- J1 pad 2: unconnected-(J1-Pin_2-Pad2) -> LED_G_OUT
- J1 pad 3: unconnected-(J1-Pin_3-Pad3) -> LED_R_OUT
- J1 pad 4: unconnected-(J1-Pin_4-Pad4) -> +12V
- R2 pad 1: unconnected-(R2-Pad1) -> Net-(U1-IO18)
- U1 pad 17: unconnected-(U1-IO19-Pad17) -> RELAY
- U1 pad 18: unconnected-(U1-IO18-Pad18) -> Net-(U1-IO18)
- U1 pad 21: LED_R -> LED_B
- U1 pad 23: LED_B -> LED_R
Routing:
- net +12V: track 46.6 -> 173.5 mm, vias 0 -> 2
- net +3V3: track 0.00 -> 102.1 mm
- net Net-(Q7-B): track 0.00 -> 49.5 mm
- net +5V: track 0.00 -> 41.8 mm
- net LED_B: track 0.00 -> 31.5 mm
- net LED_B_OUT: track 0.00 -> 23.3 mm
- net LED_G_OUT: track 0.00 -> 16.1 mm
- net LED_R_OUT: track 0.00 -> 15.5 mm
- net Net-(Q5-C): track 0.00 -> 15.3 mm
- net LED_G: track 0.00 -> 15.3 mm
- net Net-(D2-A): track 2.99 -> 17.4 mm
- net Net-(D1-A): track 2.95 -> 15.3 mm
- net Net-(Q1-G): track 0.00 -> 10.2 mm
- net Net-(Q3-C): track 0.00 -> 9.36 mm
- net Net-(Q3-B): track 0.00 -> 7.83 mm
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Other:
- board text added: "WIFI RGB and LOAD CTRL"
